Commit message: Publishing extra joints [week-1 currently working now]

File: Week-1/Challenge/Puzzlebot_Gazebo_Simulator/src/puzzlebot_gazebo/urdf/puzzlebot.xacro (robot description, xacro)
@@ -193,4 +193,9 @@
                 <state_interface name="effort"/>
               </joint>
+              <joint name="base_link_to_chassis">
+                <state_interface name="position" />
+                <state_interface name="velocity"/>
+                <state_interface name="effort"/>
+              </joint>
             </ros2_control>
           </robot>
