Commit message: Added lidar. Bug 0 WIP

File: Week-1/Challenge/Puzzlebot_Gazebo_Simulator/src/puzzlebot_gazebo/urdf/parameters.xacro (robot description, xacro)
@@ -22,3 +22,4 @@
 <xacro:property name="mesh_wheel"  value="$(find puzzlebot_gazebo)/meshes/wheel.stl" />
 <xacro:property name="mesh_camera"  value="$(find puzzlebot_gazebo)/meshes/camera.stl" />
+<xacro:property name="mesh_lidar"  value="$(find puzzlebot_gazebo)/meshes/lidar.stl" />
 </robot>

File: Week-1/Challenge/Puzzlebot_Gazebo_Simulator/src/puzzlebot_gazebo/urdf/puzzlebot.xacro (robot description, xacro)
@@ -133,4 +133,24 @@
           </visual>
         </link>
+        <!-- LIDAR-->
+        <link name="lidar">
+          <inertial>
+            <mass value="0.1" />
+            <origin xyz="0 0 0" />
+            <inertia ixx="0.01" ixy="0.0" ixz="0.0" iyy="0.01" iyz="0.0" izz="0.01" />
+          </inertial>
+          <collision>
+            <origin xyz="-0.06 0.0 -0.04" rpy="0 0 0" />
+            <geometry>
+              <cylinder length="0.01" radius="0.05"/>
+            </geometry>
+          </collision>
+          <visual>
+            <origin rpy="${PI/2} 0 0" xyz="0.07 -0.013 -0.04" />
+            <geometry>
+              <mesh filename="file://${mesh_lidar}" />
+            </geometry>
+          </visual>
+        </link>
         <!-- JOINTS  -->
         <joint name="base_to_right_w" type="continuous">
@@ -156,4 +176,9 @@
               <origin xyz="0.09 0 0.048" rpy= "0.0 0.24 0.0" />
             </joint>
+            <joint name="lidar_to_base" type="fixed">
+              <parent link="chassis"/>
+              <child link="lidar"/>
+              <origin xyz="0.05 0 0.115" rpy="0 0 ${PI}"/>
+            </joint>
             <!-- TRANSMISSIONS (For a more complex model and it represents actuator attributes) -->
             <transmission name="right_wheel_trans">
